Commit message: added basic simulation functionality with manual drive controls

File: description/robot_core.xacro (robot description, xacro)
@@ -4,4 +4,5 @@
     <link name="base_link">
     </link>
+    <!-- CHASSIS -->
     <joint name="chassis_joint" type="fixed">
         <parent link="base_link"/>
@@ -27,4 +28,7 @@
         </xacro:inertial_box>
     </link>
+    <gazebo reference="chassis">
+        <material>Gazebo/White</material>
+    </gazebo>
     <!-- LEFT WHEEL -->
     <joint name="left_wheel_joint" type="continuous">
@@ -50,4 +54,7 @@
         </xacro:inertial_cylinder>
     </link>
+    <gazebo reference="left_wheel">
+        <material>Gazebo/Blue</material>
+    </gazebo>
     <!-- RIGHT WHEEL -->
     <joint name="right_wheel_joint" type="continuous">
@@ -62,4 +69,5 @@
                 <cylinder length="0.04" radius="0.05" />
             </geometry>
+            <material name="blue"/>
         </visual>
         <collision>
@@ -72,4 +80,7 @@
         </xacro:inertial_cylinder>
     </link>
+    <gazebo reference="right_wheel">
+        <material>Gazebo/Blue</material>
+    </gazebo>
     <!-- CASTER WHEEL -->
     <joint name="caster_wheel_joint" type="fixed">
@@ -94,4 +105,10 @@
         </xacro:inertial_sphere>
     </link>
+    <gazebo reference="caster_wheel">
+        <material>Gazebo/Black</material>
+        <mu1 value="0.001"/>
+        <mu2 value="0.001"/>
+    </gazebo>
+    <!-- MATERIALS -->
     <material name="white">
         <color rgba="1 1 1 1"/>

Commit message: hopeless lidar simulation attempts

File: description/robot_core.xacro (robot description, xacro)
@@ -123,3 +123,6 @@
         <color rgba="0 0 0 1"/>
     </material>
+    <material name="red">
+        <color rgba="1 0 0 1"/>
+    </material>
 </robot>
