Commit message: lidar simulation now works and publishes data to /scan topic

File: description/lidar.xacro (robot description, xacro)
@@ -1,10 +1,10 @@
 <?xml version="1.0"?>
 <robot xmlns:xacro="http://www.ros.org/wiki/xacro">
-    <joint name="lidar_joint" type="fixed">
+    <joint name="laser_joint" type="fixed">
         <parent link="base_link"/>
-        <child link="lidar_link"/>
+        <child link="laser_frame"/>
         <origin xyz="-0.05 0 0.175" rpy="0 0 0"/>
     </joint>
-    <link name="lidar_link">
+    <link name="laser_frame">
         <visual>
             <geometry>
@@ -22,6 +22,27 @@
         </xacro:inertial_cylinder>
     </link>
-    <gazebo reference="laser_frame">
-        <material>Gazebo/Red</material>
-    </gazebo>
+ <gazebo reference="laser_frame">
+    <material>Gazebo/Red</material>
+    <sensor name="laser" type="gpu_lidar">
+         <pose> 0 0 0 0 0 0 </pose>
+         <always_on>true</always_on>
+         <visualize>true</visualize>
+         <update_rate>10</update_rate>
+         <topic>scan</topic>
+         <gz_frame_id>laser_frame</gz_frame_id>
+         <lidar>
+            <scan>
+               <horizontal>
+               <samples>360</samples>
+               <min_angle>-3.14</min_angle>
+               <max_angle>3.14</max_angle>
+               </horizontal>
+            </scan>
+            <range>
+               <min>0.3</min>
+               <max>12</max>
+            </range>
+         </lidar>
+      </sensor>
+</gazebo>
 </robot>
